File: Spark.sch (EAGLE design)
At the start: 3 parts

Commit message: thermometer interface
Parts:
- added JP2: (no value), pinhead:PINHD-1X4
Connections:
- new net 3.3V: JP2.3
- new net RX: JP2.2
- new net TX: JP2.1
- net GND: now also JP2.4
Changed lines of the file:
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@@
 <part name="JP1" library="SparkFun-Connectors" deviceset="M02" device="5MM"/>
 <part name="P+1" library="supply1" deviceset="VCC" device=""/>
+<part name="JP2" library="pinhead" deviceset="PINHD-1X4" device=""/>
+<part name="GND3" library="supply1" deviceset="GND" device=""/>
+<part name="SUPPLY1" library="SparkFun-Aesthetics" deviceset="3.3V" device=""/>
 </parts>
 <sheets>
@@
 <instance part="JP1" gate="G$1" x="45.72" y="45.72" rot="R270"/>
 <instance part="P+1" gate="VCC" x="55.88" y="35.56" rot="R270"/>
+<instance part="JP2" gate="A" x="83.82" y="43.18"/>
+<instance part="GND3" gate="1" x="71.12" y="35.56"/>
+<instance part="SUPPLY1" gate="G$1" x="68.58" y="43.18" rot="R90"/>
 </instances>
 <busses>
@@
 <wire x1="45.72" y1="25.4" x2="45.72" y2="22.86" width="0.1524" layer="91"/>
 </segment>
+<segment>
+<pinref part="JP2" gate="A" pin="4"/>
+<wire x1="81.28" y1="40.64" x2="71.12" y2="40.64" width="0.1524" layer="91"/>
+<pinref part="GND3" gate="1" pin="GND"/>
+<wire x1="71.12" y1="40.64" x2="71.12" y2="38.1" width="0.1524" layer="91"/>
+</segment>
 </net>
 <net name="VCC" class="0">
@@
 </segment>
 </net>
+<net name="TX" class="0">
+<segment>
+<pinref part="JP2" gate="A" pin="1"/>
+<wire x1="81.28" y1="48.26" x2="73.66" y2="48.26" width="0.1524" layer="91"/>
+<label x="73.66" y="48.26" size="1.016" layer="95" rot="R180" xref="yes"/>
+</segment>
+</net>
+<net name="RX" class="0">
+<segment>
+<pinref part="JP2" gate="A" pin="2"/>
+<wire x1="81.28" y1="45.72" x2="73.66" y2="45.72" width="0.1524" layer="91"/>
+<label x="73.66" y="45.72" size="1.016" layer="95" rot="R180" xref="yes"/>
+</segment>
+</net>
+<net name="3.3V" class="0">
+<segment>
+<pinref part="JP2" gate="A" pin="3"/>
+<wire x1="81.28" y1="43.18" x2="68.58" y2="43.18" width="0.1524" layer="91"/>
+<pinref part="SUPPLY1" gate="G$1" pin="3.3V"/>
+</segment>
+</net>

Commit message: teensy
Parts:
- added JP3: (no value), pinhead:PINHD-1X4
- added JP4: (no value), pinhead:PINHD-1X3
- added JP5: (no value), SparkFun-Connectors:M025MM
- added U$1: TEENSY_3.1_BASIC, Teensy_3_Series_Board_v1.0:TEENSY_3.1_BASIC
Connections:
- new net CLK: JP3.3, U$1.3/CAN-TX/PWM
- new net DAT: JP3.2, U$1.2
- new net TX2: JP4.3, U$1.10/TX2/PWM
- net 3.3V: now also JP3.1, JP4.1, U$1.3.3V
- net GND: now also JP3.4, JP4.2, JP5.2, U$1.GND
- net IGNITE: now also U$1.4/CAN-RX-PWM
- net RX: now also U$1.0/RX1/T
- net TX: now also U$1.1/TX1/T
- net VCC: now also JP5.1
Other:
- moved on the sheet: JP1, JP2, Q1, R1
